File: ion-xgt-adapter/ion-connector-bottom.kicad_sch (KiCad schematic)
At the start: 12 parts

Commit message: Working version
Parts:
- removed HALL1: Conn_01x05, Connector_Molex:Molex_KK-254_AE-6410-05A_1x05_P2.54mm_Vertical, symbol Connector_Generic:Conn_01x05
- removed PhG1: Conn_01x02, TerminalBlock_WAGO:TerminalBlock_WAGO_236-402_1x02_P5.00mm_45Degree, symbol Connector_Generic:Conn_01x02
- added B2B1: Conn_02x03_Odd_Even, Connector_PinHeader_2.54mm:PinHeader_2x03_P2.54mm_Vertical, symbol Connector_Generic:Conn_02x03_Odd_Even
- added J1: Conn_01x06, Connector_Molex:Molex_KK-254_AE-6410-06A_1x06_P2.54mm_Vertical, symbol Connector_Generic:Conn_01x06
- added J2: Conn_01x01, TerminalBlock_WAGO:TerminalBlock_WAGO_236-401_1x01_P5.00mm_45Degree, symbol Connector_Generic:Conn_01x01
- added TEMP/RPM1: Conn_01x03, Connector_Molex:Molex_KK-254_AE-6410-03A_1x03_P2.54mm_Vertical, symbol Connector_Generic:Conn_01x03
- H1, H2, H3: footprint MountingHole:MountingHole_3.2mm_M3_DIN965_Pad -> Library:MountingHole_3.6mm_M3_DIN965_Pad
- renumbered HG1 to HB1, HY1 to HG1, HB1 to HY1, PhYB1 to Ph1
Connections:
- net +5V: now also B2B1.1 (Pin_1), J1.1 (Pin_1), TEMP/RPM1.1 (Pin_1)
- net G: now also J2.1 (Pin_1)
- net GND: now also B2B1.2 (Pin_2), J1.2 (Pin_2), TEMP/RPM1.2 (Pin_2)
- net HY: now reaches HY1.3 (Pin_3)
- net HY: now also B2B1.4 (Pin_4), J1.4 (Pin_4)
- net HB: now reaches HB1.3 (Pin_3)
- net HB: now also B2B1.5 (Pin_5), J1.5 (Pin_5)
- net HG: now reaches HG1.3 (Pin_3)
- net HG: now also B2B1.3 (Pin_3), J1.3 (Pin_3)
- new net TEMP: B2B1.6 (Pin_6), J1.6 (Pin_6), TEMP/RPM1.3 (Pin_3)
